File: hardware/akaLinkCompact.kicad_pcb (KiCad board)
At the start: 2 copper layers, 45 x 45 mm, 57 parts, among them J101 USB_C_Receptacle, J102 IDC_20P, Q104 AO3400A, U101 XC6206P332MR, U102 CH32V30xFxPx, U103 SN74LVC1T45DBV, U104 USBLC6-2SC6, U105 TPS22918DBV, U110 SN74LVC1T45DBV, U111 SN74LVC1T45DBV, U112 SN74LVC1T45DBV, U113 SN74LVC1T45DBV, Y101 12MHz

Commit message: add hardware
Parts:
- U102: value CH32V30xFxPx -> CH32V305FBP6
- moved C118 0.10 mm to (85.5, 90.2)
Routing:
- net GND: vias 35 -> 46
Other:
- board text added: "SWD+VCOM"
- board text added: "akaLink Compact Rev A.1 @2026/03/14"
- board text removed: "SWD"
