File: hardware/akaLinkCompact.kicad_sch (KiCad schematic)
At the start: 57 parts, among them J101 USB_C_Receptacle, J102 IDC_20P, Q104 AO3400A, U101 XC6206P332MR, U102 CH32V30xFxPx, U103 SN74LVC1T45DBV, U104 USBLC6-2SC6, U105 TPS22918DBV, U110 SN74LVC1T45DBV, U111 SN74LVC1T45DBV, U112 SN74LVC1T45DBV, U113 SN74LVC1T45DBV, Y101 12MHz

Commit message: add hardware
Parts:
- U102: value CH32V30xFxPx -> CH32V305FBP6
Other:
- note added: "UART3_RX"
- note added: "UART3_TX"
- note removed: "Sense"
- moved on the sheet: C103, Q104, R117, R124, R125, R133
